Commit message: fix some error in urdf and add rplidar dae file

File: bada_g2_description/urdf/bada_g2.xacro (robot description, xacro)
@@ -176,5 +176,5 @@
       <origin xyz="0 0 -0.0308" rpy="1.5707 0 4.71"/>
       <geometry>
-        <mesh filename="package://my_mobile/meshes/rplidar.dae" scale="0.001 0.001 0.001" />
+        <mesh filename="package://bada_g2_description/meshes/rplidar.dae" scale="0.001 0.001 0.001" />
       </geometry>
     </collision>
@@ -182,5 +182,5 @@
       <origin xyz="0 0 -0.0308" rpy="1.5707 0 4.71"/>
       <geometry>
-        <mesh filename="package://my_mobile/meshes/rplidar.dae" scale="0.001 0.001 0.001" />
+        <mesh filename="package://bada_g2_description/meshes/rplidar.dae" scale="0.001 0.001 0.001" />
       </geometry>
     </visual>

File: bada_g2_description/urdf/bada_g2_description.urdf (robot description, URDF)
Before this commit: robot bada_g2_description, 5 links, 4 joints
Links:
- link laser: geometry collision mesh filename=package://bada_g2_description/meshes/rplidar.dae scale=0.001 0.001 0.001; visual mesh filename=package://bada_g2_description/meshes/rplidar.dae scale=0.001 0.001 0.001

Commit message: update for real world bada robot

File: bada_g2_description/urdf/bada_g2.xacro (robot description, xacro)
@@ -168,5 +168,5 @@
   <joint name="rplidar_joint" type="fixed">
     <axis xyz="0 1 0" />
-    <origin xyz="0.145 0 0.085" rpy="0 0 0"/> <!--rpy : 0 0 3.14-->
+    <origin xyz="0.145 0 0.085" rpy="0 0 -3.14"/> <!--simulation rpy : 0 0 0-->
     <parent link="base_link"/>
     <child link="laser"/>

Commit message: update for real world and simulation version

File: bada_g2_description/urdf/bada_g2.xacro (robot description, xacro)
@@ -168,6 +168,6 @@
   <joint name="rplidar_joint" type="fixed">
     <axis xyz="0 1 0" />
-    <origin xyz="0.145 0 0.085" rpy="0 0 -3.14"/> <!--simulation rpy : 0 0 0-->
-    <parent link="base_link"/>
+    <origin xyz="0.145 0 0.085" rpy="0 0 0"/> <!--simulation rpy : 0 0 0-->
+    <parent link="base_link"/>                    <!--real world rpy : 0 0 -3.14-->
     <child link="laser"/>
   </joint>
